File: electronics/kicad/fd1_controller.kicad_sch (KiCad schematic)
At the start: 44 parts, among them J1 USB D-/D+ (native USB), J10 Throttle servo, J11 Servo 6 V BEC in, J12 3-way router valve, J13 Stack light + buzzer, J14 microSD module, J15 12 V DC in, J16 EN / BOOT / GND, J2 SDP810-500Pa dP, J3 SHT40 T/RH, J4 SEN0322 O2, J5 SSD1306 OLED, J6 MH-440D CH4 NDIR, J7 MPX5100AP pressure, J8 RS-485 to gateway, J9 NC solenoid 12 V, Q1 IRLZ44N, U1 ESP32-S3-WROOM-1-N8R8, U2 MAX3485, U3 DRV8871, U4 ULN2003A, U5 MP1584 buck module 12V>5V, U6 AMS1117-3.3

Commit message: PCB layout + DRC, low-cost BOM with price basis, team names, deck v3
- electronics/kicad: routed 2-layer PCB (110x80 mm), DRC 0 errors, renders, stats
- electronics/bom.py: Stage 3 build Rs 48,400 with a price source per line
- docs: sources, references, glossary; README updated

Co-Authored-By: Claude Opus 5.5 <noreply@anthropic.com>
Claude-Session: https://claude.ai/code/session_01Vz7JfuGgWMU6CCjesC947p
Parts:
- U2: footprint (none) -> Package_SO:SOIC-8_3.9x4.9mm_P1.27mm
- U4: footprint (none) -> Package_DIP:DIP-16_W7.62mm
Changed lines of the file:
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@@
   (property "Reference" "U2" (at 299.72 35.56 0) (effects (font (size 1.27 1.27))))
   (property "Value" "MAX3485" (at 299.72 43.18 0) (effects (font (size 1.27 1.27))))
-  (property "Footprint" "" (at 299.72 39.37 0) (effects (font (size 1.27 1.27)) hide))
+  (property "Footprint" "Package_SO:SOIC-8_3.9x4.9mm_P1.27mm" (at 299.72 39.37 0) (effects (font (size 1.27 1.27)) hide))
   (property "Datasheet" "https://datasheets.maximintegrated.com/en/ds/MAX3483-MAX3491.pdf" (at 299.72 39.37 0) (effects (font (size 1.27 1.27)) hide))
   (pin "1")
@@
   (property "Reference" "U4" (at 299.72 226.06 0) (effects (font (size 1.27 1.27))))
   (property "Value" "ULN2003A" (at 299.72 233.68 0) (effects (font (size 1.27 1.27))))
-  (property "Footprint" "" (at 299.72 229.87 0) (effects (font (size 1.27 1.27)) hide))
+  (property "Footprint" "Package_DIP:DIP-16_W7.62mm" (at 299.72 229.87 0) (effects (font (size 1.27 1.27)) hide))
   (property "Datasheet" "http://www.ti.com/lit/ds/symlink/uln2003a.pdf" (at 299.72 229.87 0) (effects (font (size 1.27 1.27)) hide))
   (pin "1")
